File: Electronics/RFID_Extension/RFID_Extension.kicad_sch (KiCad schematic)
At the start: 1 part, among them U1 ESP32-C3-WROOM-02

Commit message: 最低限の回路作製
Parts:
- added C1: 0.1u, symbol Device:C_Small
- added C2: 4u7, symbol Device:C_Small
- added C3, C4: 1u, symbol Device:C_Small
- added D1, D2: LED, symbol Device:LED
- added D1_POW: G, symbol Device:LED
- added F1: Fuse, symbol Device:Fuse
- added J1_I2C, J1_Write: PinHeader, symbol Connector:Conn_01x04_Pin
- added J1_POWER: XT, symbol Connector:Conn_01x02_Socket
- added Q1, Q2: NPN, symbol Simulation_SPICE:NPN
- added R1, R3: 47k, symbol Device:R_Small
- added R2, R4: 1k, symbol Device:R_Small
- added RN1, RN2: 10k, symbol Device:R_Pack04
- added U2: AP7381-33SA-7, Package_TO_SOT_SMD:SOT-23, symbol Regulator_Linear:AP7381-33SA-7
Connections:
- net +3V3: now reaches U1.1 (3V3)
- net +3V3: now also U1.2 (EN), C1.1, C2.1, C4.1, J1_I2C.2 (Pin_2), J1_Write.2 (Pin_2), R2.1, R4.1, RN1.5 (R4.2), RN1.6 (R3.2), RN1.7 (R2.2), RN1.8 (R1.2), RN2.5 (R4.2), RN2.6 (R3.2), RN2.7 (R2.2), RN2.8 (R1.2), U2.2 (VO)
- net RX: now reaches U1.11 (IO20/RXD)
- net RX: now also J1_Write.3 (Pin_3)
- net TX: now reaches U1.12 (IO21/TXD)
- net TX: now also J1_Write.4 (Pin_4)
- net GND: now reaches U1.19 (GND), U1.9 (GND)
- net GND: now also C1.2, C2.2, C3.2, C4.2, D1_POW.1 (K), J1_I2C.1 (Pin_1), J1_POWER.1 (Pin_1), J1_Write.1 (Pin_1), Q1.3 (E), Q2.3 (E), U2.3 (GND)
- net SDA: now reaches U1.3 (IO4)
- net SDA: now also J1_I2C.3 (Pin_3), RN1.1 (R1.1), RN1.2 (R2.1)
- net SCL: now reaches U1.4 (IO5)
- net SCL: now also J1_I2C.4 (Pin_4), RN1.3 (R3.1), RN1.4 (R4.1)
- net USR1: now reaches U1.6 (IO7)
- net USR1: now also R1.1
- net USR2: now reaches U1.7 (IO8)
- net USR2: now also R3.1
- new net: D1.2 (A), R2.2
- new net: C3.1, F1.2, U2.1 (VI)
- new net: D2.1 (K), Q2.1 (C)
- new net: D2.2 (A), R4.2
- new net: D1.1 (K), Q1.1 (C)
- new net: Q1.2 (B), R1.2
- new net: Q2.2 (B), R3.2
- new net: D1_POW.2 (A), RN2.1 (R1.1), RN2.2 (R2.1), RN2.3 (R3.1), RN2.4 (R4.1)
- new net VCC: F1.1, J1_POWER.2 (Pin_2)
Other:
- note added: "Battery"
- note added: "I2C Connect"
- note added: "LDO"
- note added: "MCU"
- note added: "RX to TX TX to RX"
- note added: "USER LED"
- note added: "Write"
- moved on the sheet: U1
